Commit message: Upgrading while preparing next video

File: description/robot_car.urdf (robot description, URDF)
Before this commit: robot robot_car, 8 links, 7 joints
Joints:
- joint antenna_joint: origin xyz=-0.07 -${base_width/2 - antenna_width/2} ${base_height/2 + board_1_height + antenna_height/2} -> xyz=-0.06 -${base_width/2 - antenna_width/2} ${base_height/2 + board_1_height + antenna_height/2}
