Commit message: Fix physical RPLIDAR setup

File: robot_car/description/robot_car.physical.urdf (robot description, URDF)
Before this commit: robot robot_car, 8 links, 7 joints
Joints:
- joint lidar_joint: origin xyz=0.03 0.00 ${base_height/2 + tower_height + lidar_width/2} rpy=0 0 0 -> xyz=0.03 0.00 ${base_height/2 + tower_height + lidar_width/2} rpy=0 0 ${pi}
